File: PCBs/Estación terreno/Estación terreno.kicad_pcb (KiCad board)
At the start: 2 copper layers, 100 x 90 mm, 11 parts, among them U1 ESP32-DEVKIT-V1, U3 TFT_320x240

Commit message: feat: Se agrega la versión completa de la PCB y los archivos de fabricación
Parts:
- added G***: LOGO, Images:Logo-Pavo's-Robotics-Projects, F.Cu at (48.5, 60.7)
- moved U2 2.24 mm to (42.2, 32.3)
Routing:
- net 3V3: track 0.00 -> 161.2 mm, vias 0 -> 1
- net SCK: track 0.00 -> 139.1 mm, vias 0 -> 1
- net ALERTA: track 0.00 -> 128.6 mm, vias 0 -> 1
- net MISO: track 0.00 -> 110.2 mm, vias 0 -> 1
- net MOSI: track 0.00 -> 104.4 mm, vias 0 -> 1
- net MISSING: track 0.00 -> 86.8 mm, vias 0 -> 1
- net OK: track 0.00 -> 76.1 mm, vias 0 -> 1
- net LED_TFT: track 0.00 -> 73.4 mm
- net Net-(D1-A): track 0.00 -> 73.4 mm
- net RST_LORA: track 0.00 -> 66.1 mm
- net NSS_LORA: track 0.00 -> 65.4 mm
- net DIO0: track 0.00 -> 57.3 mm
- net Net-(D2-A): track 0.00 -> 56.0 mm, vias 0 -> 2
- net DC_TFT: track 0.00 -> 33.0 mm, vias 0 -> 1
- net RST_TFT: track 0.00 -> 32.7 mm
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- added copper zone on B.Cu, net GND
- added copper zone on F.Cu, net GND
Other:
- board text added: "D1"
- board text added: "D2"
- board text added: "D3"
- board text added: "D4"
- board text added: "Estación Terrena V1"
- board text added: "MISSING"
- board text added: "OK"
- board text added: "PWR"
- board text added: "WARNING"
