File: PCBs/Estación terreno/Estación terreno.kicad_sch (KiCad schematic)
At the start: 11 parts, among them U1 ESP32-DEVKIT-V1, U3 TFT_320x240

Commit message: feat: Se agrega la versión completa de la PCB y los archivos de fabricación
Connections:
- no-connect marks 0 -> 10
Changed lines of the file:
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@@
 		(color 0 0 0 0)
+	)
+	(no_connect
+		(at 168.91 71.12)
+	)
+	(no_connect
+		(at 113.03 59.69)
+	)
+	(no_connect
+		(at 171.45 71.12)
+	)
+	(no_connect
+		(at 113.03 57.15)
+	)
+	(no_connect
+		(at 90.17 59.69)
+	)
+	(no_connect
+		(at 176.53 71.12)
+	)
+	(no_connect
+		(at 90.17 57.15)
+	)
+	(no_connect
+		(at 173.99 71.12)
+	)
+	(no_connect
+		(at 179.07 71.12)
+	)
+	(no_connect
+		(at 90.17 62.23)
 	)
 	(wire
